Commit message: 

File: trunk/ros/lrm_carina/lrm_description/urdf/clubcar/stereo.camera.urdf.xacro (robot description, xacro)
@@ -54,5 +54,5 @@
 		image_topic_name="image_raw"
 		camera_info_topic_name="camera_info"
-		parent="base_front_sensors"
+		parent="base_stereo_camera"
 		hfov="43"
 		focal_length="812.366824"
@@ -72,5 +72,5 @@
 		image_topic_name="image_raw"
 		camera_info_topic_name="camera_info"
-		parent="base_front_sensors"
+		parent="base_stereo_camera"
 		hfov="43"
 		focal_length="812.366824"
@@ -108,10 +108,23 @@
 	>
 		<origin
-			xyz="-0.1 0 0.1"
+			xyz="0.0 0.0 0.12"
 			rpy="0 0 0 " />
 		<parent link="base_front_sensors" />
+		<child link="base_stereo_camera" />
+	</joint>
+	<joint
+		name="base_camera_center_joint"
+		type="fixed"
+	>
+		<origin
+			xyz="-0.1 0.0 0.1"
+			rpy="0 0 0" />
+		<parent link="base_stereo_camera" />
 		<child link="camera_center_link" />
 	</joint>
 	<link name="stereo_camera">
+		<xacro:inertial_minimal />
+	</link>
+	<link name="base_stereo_camera">
 		<xacro:inertial_minimal />
 	</link>
