Commit message: 

File: trunk/ros/lrm_carina/lrm_description/urdf/clubcar/base.urdf.xacro (robot description, xacro)
@@ -37,4 +37,7 @@
 	<link name="base_footprint" />
 	<link name="base_link">
+		<xacro:inertial_minimal />
+	</link>
+	<link name="heading_link">
 		<xacro:inertial_minimal />
 	</link>
@@ -115,4 +118,14 @@
 	</joint>
 	<joint
+		name="joint_base_heading"
+		type="fixed"
+	>
+		<origin
+			rpy="0 0 0"
+			xyz="0 0 ${-wheel_diameter/2}" />
+		<parent link="front_axle_link" />
+		<child link="heading_link" />
+	</joint>
+	<joint
 		name="joint_base_link_to_rear_axle"
 		type="fixed"

Commit message: 

File: trunk/ros/lrm_carina/lrm_description/urdf/clubcar/base.urdf.xacro (robot description, xacro)
@@ -41,4 +41,14 @@
 	<link name="heading_link">
 		<xacro:inertial_minimal />
+		<visual>
+			<geometry>
+				<cylinder
+					radius="0.03"
+					length="0.045" />
+			</geometry>
+			<material name="Red">
+				<color rgba="0.8 0.0 0.0 1.0" />
+			</material>
+		</visual>
 	</link>
 	<link name="center_mass_link">

File: trunk/ros/lrm_carina/lrm_description/urdf/clubcar/common.xacro (robot description, xacro)
@@ -82,5 +82,5 @@
 	<property
 		name="drive_torque"
-		value="99000000" /> <!--  700000    1 hp = 746 W = 746 N·m/s -> clubcar motor ~ 9.5 Hp -->
+		value="700000" /> <!--  700000    1 hp = 746 W = 746 N·m/s -> clubcar motor ~ 9.5 Hp -->
 	<property
 		name="steer_torque"
